Commit message: reorganized urdf folder, added README and optimized launch

File: urdf/wheels/caster_wheel.urdf.xacro (robot description, xacro)
@@ -1,6 +1,7 @@
 <?xml version="1.0"?>
 <robot xmlns:xacro="http://ros.org/wiki/xacro">
+  <!-- Includes -->
   <xacro:include filename="caster_wheel.gazebo.xacro"/>
-  <xacro:macro name="caster" params="name radius x_offset y_offset z_offset parent">
+  <xacro:macro name="caster_wheel" params="name radius mass x_offset y_offset z_offset parent">
     <link name="${name}_link">
       <visual>
@@ -9,5 +10,5 @@
           <sphere radius="${radius}"/>
         </geometry>
-        <material name="black"/>
+        <material name="grey"/>
       </visual>
       <collision>
@@ -19,7 +20,7 @@
       </collision>
       <inertial>
-        <origin xyz="${x_offset} 0 0" rpy="0 0 0"/>
-        <mass value="4.0"/>
-        <xacro:solid_sphere_inertia r="${radius}" m="4.0"/>
+        <origin xyz="0 0 0" rpy="0 0 0"/>
+        <mass value="${mass}"/>
+        <xacro:sphere_inertia r="${radius}" m="${mass}"/>
         <inertia />
       </inertial>
@@ -31,5 +32,5 @@
     </joint>
     <!-- Gazebo extensions -->
-    <caster_gazebo name="${name}"/>
+    <xacro:caster_wheel_gazebo name="${name}"/>
   </xacro:macro>
 </robot>
