Commit message: fixed inertia and contact model of the caster wheels

File: urdf/base/palletron_base.urdf.xacro (robot description, xacro)
@@ -7,5 +7,5 @@
   <!-- TODO: Update according to real base properties -->
   <!-- Base properties -->
-  <xacro:property name="base_mass" value="50.0"/>
+  <xacro:property name="base_mass" value="25.0"/>
   <xacro:property name="base_width" value="0.7"/>
   <xacro:property name="base_depth" value="0.7"/>
@@ -24,5 +24,5 @@
   <xacro:property name="caster_x_offset" value="0.25"/>
   <xacro:property name="caster_y_offset" value="0.25"/>
-  <xacro:property name="caster_ground_offset" value="0.0005"/>
+  <xacro:property name="caster_ground_offset" value="0.005"/>
   <!-- Base -->
   <xacro:macro name="palletron_base">

File: urdf/wheels/caster_wheel.gazebo.xacro (robot description, xacro)
@@ -8,9 +8,9 @@
       <kp>1000000.0</kp>
       <kd>100.0</kd>
-      <mu1>0.3</mu1>
-      <mu2>0.3</mu2>
+      <mu1>0.0</mu1>
+      <mu2>0.0</mu2>
       <fdir1>1 0 0</fdir1>
       <maxVel>1.0</maxVel>
-      <minDepth>0.00</minDepth>
+      <minDepth>0.0</minDepth>
       <implicitSpringDamper>1</implicitSpringDamper>
     </gazebo>

File: urdf/wheels/caster_wheel.urdf.xacro (robot description, xacro)
@@ -21,6 +21,8 @@
       <inertial>
         <origin xyz="0 0 0" rpy="0 0 0"/>
-        <mass value="${mass}"/>
-        <xacro:sphere_inertia r="${radius}" m="${mass}"/>
+        <mass value="0.005"/>
+        <inertia ixx="0.001" ixy="0" ixz="0"
+                 iyy="0.001" iyz="0"
+                 izz="0.001"/>
         <inertia />
       </inertial>
