Commit message: added namespace to the robots and reorganized urdf files (again)

File: urdf/bases/default_base.urdf.xacro (robot description, xacro)
@@ -1,13 +1,12 @@
 <?xml version="1.0"?>
 <robot xmlns:xacro="http://ros.org/wiki/xacro">
-  <xacro:include filename="default_base.gazebo.xacro"/>
-  <xacro:macro name="default_base_macro" params="mass width height depth *origin">
-    <link name="base_footprint"/>
-    <joint name="base_joint" type="fixed">
+  <xacro:macro name="default_base_macro" params="robot_namespace mass width height depth *origin">
+    <link name="${robot_namespace}/base_footprint"/>
+    <joint name="${robot_namespace}/base_joint" type="fixed">
       <xacro:insert_block name="origin"/>
-      <parent link="base_footprint"/>
-      <child link="base_link" />
+      <parent link="${robot_namespace}/base_footprint"/>
+      <child link="${robot_namespace}/base_link" />
     </joint>
-    <link name="base_link">
+    <link name="${robot_namespace}/base_link">
       <visual>
         <origin xyz="0 0 0" rpy="0 0 0"/>
@@ -29,6 +28,18 @@
       </inertial>
     </link>
-    <!-- Include Gazebo extensions -->
-    <xacro:default_base_gazebo_macro/>
+    <!-- Gazebo extensions -->
+    <gazebo reference="${robot_namespace}/base_link">
+      <material>Gazebo/Blue</material>
+    </gazebo>
+    <gazebo reference="${robot_namespace}/base_footprint">
+      <kp>100000000.0</kp>
+      <kd>10.0</kd>
+      <mu1>0.1</mu1>
+      <mu2>0.1</mu2>
+      <fdir1>1 0 0</fdir1>
+      <maxVel>10.0</maxVel>
+      <minDepth>0.0005</minDepth>
+      <laserRetro>0</laserRetro>
+    </gazebo>
   </xacro:macro>
 </robot>

File: urdf/controllers/differential_drive.gazebo.xacro (robot description, xacro)
@@ -1,26 +1,26 @@
 <?xml version="1.0"?>
 <robot xmlns:xacro="http://ros.org/wiki/xacro">
-  <xacro:macro name="differential_drive_macro" params="right_wheel_prefix left_wheel_prefix wheel_separation wheel_diameter wheel_max_torque wheel_max_acceleration">
+  <xacro:macro name="differential_drive_macro" params="robot_namespace right_wheel_prefix left_wheel_prefix wheel_separation wheel_diameter wheel_max_torque wheel_max_acceleration">
     <gazebo>
       <plugin name="gazebo_ros_diff_drive" filename="libgazebo_ros_diff_drive.so">
-        <odometry_topic>odom</odometry_topic>
-        <odometry_frame>odom</odometry_frame>
+        <odometry_topic>${robot_namespace}/odometry/odom_unfiltered</odometry_topic>
+        <odometry_frame>${robot_namespace}/odom</odometry_frame>
         <update_rate>30</update_rate>
-        <left_joint>${left_wheel_prefix}_joint</left_joint>
-        <right_joint>${right_wheel_prefix}_joint</right_joint>
+        <left_joint>${robot_namespace}/${left_wheel_prefix}_joint</left_joint>
+        <right_joint>${robot_namespace}/${right_wheel_prefix}_joint</right_joint>
         <wheel_separation>${wheel_separation}</wheel_separation>
         <wheel_diameter>${wheel_diameter}</wheel_diameter>
         <max_wheel_torque>${wheel_max_torque}</max_wheel_torque>
         <max_wheel_acceleration>${wheel_max_acceleration}</max_wheel_acceleration>
-        <command_topic>cmd_vel</command_topic>
+        <command_topic>${robot_namespace}/velocity_cmd</command_topic>
         <publish_odom>true</publish_odom>
         <publish_odom_tf>true</publish_odom_tf>
         <publish_wheel_tf>false</publish_wheel_tf>
-        <robot_base_frame>base_footprint</robot_base_frame>
+        <robot_base_frame>${robot_namespace}/base_footprint</robot_base_frame>
       </plugin>
       <plugin name="gazebo_ros_joint_state_publisher" filename="libgazebo_ros_joint_state_publisher.so">
         <update_rate>30</update_rate>
-        <joint_name>${right_wheel_prefix}_joint</joint_name>
-        <joint_name>${left_wheel_prefix}_joint</joint_name>
+        <joint_name>${robot_namespace}/${right_wheel_prefix}_joint</joint_name>
+        <joint_name>${robot_namespace}/${left_wheel_prefix}_joint</joint_name>
       </plugin>
     </gazebo>

File: urdf/inertias.urdf.xacro (robot description, xacro)
@@ -10,14 +10,14 @@
   <xacro:macro name="solid_cylinder_inertia_macro" params="mass radius height">
     <inertia
-      ixx="${mass * 3 * radius * radius + height * height / 12}"
-      iyy="${mass * 3 * radius * radius + height * height / 12}"
-      izz="${mass * radius * radius / 2}"
+      ixx="${mass / 12 * (3 * radius * radius + height * height)}"
+      iyy="${mass / 12 * (3 * radius * radius + height * height)}"
+      izz="${mass / 2 * (radius * radius)}"
       ixy="0" ixz="0" iyz="0"/>
   </xacro:macro>
   <xacro:macro name="solid_cuboid_inertia_macro" params="mass height depth width">
     <inertia
-      ixx="${mass * (height * height + depth * depth) / 12}"
-      iyy="${mass * (width * width + depth * depth) / 12}"
-      izz="${mass * (width * width + height * height) / 12}"
+      ixx="${mass / 12 * (height * height + depth * depth)}"
+      iyy="${mass / 12 * (width * width + depth * depth)}"
+      izz="${mass / 12 * (width * width + height * height)}"
       ixy="0" ixz="0" iyz="0"/>
   </xacro:macro>

File: urdf/palletron.xacro (robot description, xacro)
@@ -9,6 +9,8 @@
   <xacro:include filename="wheels/caster_wheel.urdf.xacro"/>
   <xacro:include filename="sensors/rplidar.urdf.xacro"/>
-  <!-- Args -->
-  <xacro:arg name="use_less_scan_samples" default="false"/>
+  <!-- Load optional properties files -->
+  <xacro:property name="namespace" value="$(arg namespace)" />
+  <xacro:property name="optional_properties" value="$(arg optional_properties)"/>
+  <xacro:property name="optionals" value="${xacro.load_yaml(optional_properties)}"/>
   <!-- TODO: Update according to real properties -->
   <!-- Base parameters -->
@@ -16,5 +18,5 @@
   <xacro:property name="base_height" value="0.7"/>
   <xacro:property name="base_depth" value="0.7"/>
-  <xacro:property name="base_mass" value="50"/>
+  <xacro:property name="base_mass" value="100"/>
   <!-- Drive wheels parameters -->
   <xacro:property name="drive_wheel_mass" value="4.0"/>
@@ -34,5 +36,6 @@
   <xacro:property name="caster_offset_ground" value="0.005"/>
   <!-- Add default base -->
-  <xacro:default_base_macro mass="${base_mass}"
+  <xacro:default_base_macro robot_namespace="${namespace}"
+    mass="${base_mass}"
     width="${base_width}"
     height="${base_height}"
@@ -42,5 +45,6 @@
   </xacro:default_base_macro>
   <!-- Add the differential drive plugin -->
-  <xacro:differential_drive_macro right_wheel_prefix="${right_drive_wheel_prefix}"
+  <xacro:differential_drive_macro robot_namespace="${namespace}"
+    right_wheel_prefix="${right_drive_wheel_prefix}"
     left_wheel_prefix="${left_drive_wheel_prefix}"
     wheel_separation="${drive_wheel_separation}"
@@ -49,6 +53,7 @@
     wheel_max_acceleration="${drive_wheel_max_acceleration}">
   </xacro:differential_drive_macro>
-  <!-- Add two drive wheels {-->
-  <xacro:drive_wheel_macro prefix="${right_drive_wheel_prefix}"
+  <!-- Add two drive wheels -->
+  <xacro:drive_wheel_macro robot_namespace="${namespace}"
+    prefix="${right_drive_wheel_prefix}"
     mass="${drive_wheel_mass}"
     radius="${drive_wheel_radius}"
@@ -57,5 +62,6 @@
     <origin xyz="0 ${-drive_wheel_separation/2} ${drive_wheel_offset_z}" rpy="${-pi/2} 0 0"/>
   </xacro:drive_wheel_macro>
-  <xacro:drive_wheel_macro prefix="${left_drive_wheel_prefix}"
+  <xacro:drive_wheel_macro robot_namespace="${namespace}"
+    prefix="${left_drive_wheel_prefix}"
     mass="${drive_wheel_mass}"
     radius="${drive_wheel_radius}"
@@ -65,5 +71,6 @@
   </xacro:drive_wheel_macro>
   <!-- Add four caster wheels -->
-  <xacro:caster_wheel_macro prefix="front_right_caster"
+  <xacro:caster_wheel_macro robot_namespace="${namespace}"
+    prefix="front_right_caster"
     mass="${caster_mass}"
     radius="${caster_radius}"
@@ -71,5 +78,6 @@
     <origin xyz="-${caster_offset_x} ${caster_offset_y} ${drive_wheel_offset_z + caster_offset_ground - (drive_wheel_radius - caster_radius)}" rpy="0 0 0"/>
   </xacro:caster_wheel_macro>
-  <xacro:caster_wheel_macro prefix="front_left_caster"
+  <xacro:caster_wheel_macro robot_namespace="${namespace}"
+    prefix="front_left_caster"
     mass="${caster_mass}"
     radius="${caster_radius}"
@@ -77,5 +85,6 @@
     <origin xyz="${caster_offset_x} ${caster_offset_y} ${drive_wheel_offset_z + caster_offset_ground - (drive_wheel_radius - caster_radius)}" rpy="0 0 0"/>
   </xacro:caster_wheel_macro>
-  <xacro:caster_wheel_macro prefix="rear_right_caster"
+  <xacro:caster_wheel_macro robot_namespace="${namespace}"
+    prefix="rear_right_caster"
     mass="${caster_mass}"
     radius="${caster_radius}"
@@ -83,5 +92,6 @@
     <origin xyz="-${caster_offset_x} -${caster_offset_y} ${drive_wheel_offset_z + caster_offset_ground - (drive_wheel_radius - caster_radius)}" rpy="0 0 0"/>
   </xacro:caster_wheel_macro>
-  <xacro:caster_wheel_macro prefix="rear_left_caster"
+  <xacro:caster_wheel_macro robot_namespace="${namespace}"
+    prefix="rear_left_caster"
     mass="${caster_mass}"
     radius="${caster_radius}"
@@ -90,5 +100,6 @@
   </xacro:caster_wheel_macro>
   <!-- Add a RPlidar -->
-  <xacro:rplidar_macro x="0"
+  <xacro:rplidar_macro robot_namespace="${namespace}"
+    x="0"
     y="0"
     z="${base_height / 2}"
@@ -96,6 +107,5 @@
     pitch="0"
     yaw="0"
-    parent="base_link"
-    use_less_scan_samples="$(arg use_less_scan_samples)">
+    parent="base_link">
   </xacro:rplidar_macro>
 </robot>

File: urdf/sensors/rplidar.urdf.xacro (robot description, xacro)
@@ -1,12 +1,11 @@
 <?xml version="1.0"?>
 <robot xmlns:xacro="http://ros.org/wiki/xacro">
-  <xacro:include filename="rplidar.gazebo.xacro"/>
-  <xacro:macro name="rplidar_macro" params="x y z roll pitch yaw parent use_less_scan_samples">
-    <joint name="rplidar_joint" type="fixed">
+  <xacro:macro name="rplidar_macro" params="robot_namespace x y z roll pitch yaw parent">
+    <joint name="${robot_namespace}/rplidar_joint" type="fixed">
       <origin xyz="${x} ${y} ${z + 0.031}" rpy="${roll} ${pitch} ${yaw}"/>
-      <parent link="${parent}"/>
-      <child link="rplidar_link"/>
+      <parent link="${robot_namespace}/${parent}"/>
+      <child link="${robot_namespace}/rplidar_link"/>
     </joint>
-    <link name="rplidar_link">
+    <link name="${robot_namespace}/rplidar_link">
       <visual>
         <origin xyz="0 0 -0.031" rpy="0 0 ${pi}"/>
@@ -18,6 +17,47 @@
       </visual>
     </link>
-    <!-- Include Gazebo extensions -->
-    <xacro:rplidar_gazebo_macro/>
+    <!-- Gazebo extensions -->
+    <gazebo reference="${robot_namespace}/rplidar_link">
+      <material>Gazebo/FlatBlack</material>
+    </gazebo>
+    <gazebo reference="${robot_namespace}/rplidar_link">
+      <sensor name="${robot_namespace}/rplidar" type="ray">
+        <always_on>true</always_on>
+        <visualize>false</visualize>
+        <update_rate>15</update_rate>
+        <ray>
+          <scan>
+            <horizontal>
+              <xacro:if value="${optionals['use_less_scan_samples']}">
+                <samples>180</samples>
+              </xacro:if>
+              <xacro:unless value="${optionals['use_less_scan_samples']}">
+                <samples>${16000/15}</samples>
+              </xacro:unless>
+              <resolution>1</resolution>
+              <min_angle>-3.1241390751</min_angle>
+              <max_angle>3.1241390751</max_angle>
+            </horizontal>
+          </scan>
+          <range>
+            <min>0.2</min>
+            <max>12</max>
+            <resolution>0.01</resolution>
+          </range>
+          <noise>
+            <type>gaussian</type>
+            <mean>0.0</mean>
+            <stddev>0.01</stddev>
+          </noise>
+        </ray>
+        <plugin name="gazebo_ros_ray_sensor" filename="libgazebo_ros_ray_sensor.so">
+          <ros>
+            <remapping>~/out:=/${robot_namespace}/rplidar/scan</remapping>
+          </ros>
+          <frame_name>${robot_namespace}/rplidar_link</frame_name>
+          <output_type>sensor_msgs/LaserScan</output_type>
+        </plugin>
+      </sensor>
+    </gazebo>
   </xacro:macro>
 </robot>

File: urdf/wheels/caster_wheel.urdf.xacro (robot description, xacro)
@@ -1,7 +1,6 @@
 <?xml version="1.0"?>
 <robot xmlns:xacro="http://ros.org/wiki/xacro">
-  <xacro:include filename="caster_wheel.gazebo.xacro"/>
-  <xacro:macro name="caster_wheel_macro" params="prefix mass radius parent *origin">
-    <link name="${prefix}_link">
+  <xacro:macro name="caster_wheel_macro" params="robot_namespace prefix mass radius parent *origin">
+    <link name="${robot_namespace}/${prefix}_link">
       <visual>
         <origin xyz="0 0 0" rpy="0 0 0"/>
@@ -23,11 +22,21 @@
       </inertial>
     </link>
-    <joint name="${prefix}_joint" type="fixed">
+    <joint name="${robot_namespace}/${prefix}_joint" type="fixed">
       <xacro:insert_block name="origin"/>
-      <parent link="${parent}"/>
-      <child link="${prefix}_link"/>
+      <parent link="${robot_namespace}/${parent}"/>
+      <child link="${robot_namespace}/${prefix}_link"/>
     </joint>
-    <!-- Include Gazebo extensions -->
-    <xacro:caster_wheel_gazebo_macro/>
+    <!-- Gazebo extensions -->
+    <gazebo reference="${robot_namespace}/${prefix}_link">
+      <material>Gazebo/Grey</material>
+      <kp>1000000.0</kp>
+      <kd>100.0</kd>
+      <mu1>0.0</mu1>
+      <mu2>0.0</mu2>
+      <fdir1>1 0 0</fdir1>
+      <maxVel>1.0</maxVel>
+      <minDepth>0.0</minDepth>
+      <implicitSpringDamper>1</implicitSpringDamper>
+    </gazebo>
   </xacro:macro>
 </robot>

File: urdf/wheels/drive_wheel.urdf.xacro (robot description, xacro)
@@ -1,7 +1,6 @@
 <?xml version="1.0"?>
 <robot xmlns:xacro="http://ros.org/wiki/xacro">
-  <xacro:include filename="drive_wheel.gazebo.xacro"/>
-  <xacro:macro name="drive_wheel_macro" params="prefix mass radius length parent *origin">
-    <link name="${prefix}_link">
+  <xacro:macro name="drive_wheel_macro" params="robot_namespace prefix mass radius length parent *origin">
+    <link name="${robot_namespace}/${prefix}_link">
       <visual>
         <origin xyz="0 0 0" rpy="0 0 0"/>
@@ -23,12 +22,22 @@
       </inertial>
     </link>
-    <joint name="${prefix}_joint" type="continuous">
+    <joint name="${robot_namespace}/${prefix}_joint" type="continuous">
       <xacro:insert_block name="origin"/>
-      <parent link="${parent}"/>
-      <child link="${prefix}_link"/>
+      <parent link="${robot_namespace}/${parent}"/>
+      <child link="${robot_namespace}/${prefix}_link"/>
       <axis xyz="0 0 1"/>
     </joint>
-    <!-- Include Gazebo extensions -->
-    <xacro:drive_wheel_gazebo_macro/>
+    <!-- Gazebo extensions -->
+    <gazebo reference="${robot_namespace}/${prefix}_link">
+      <material>Gazebo/Black</material>
+      <kp>100000.0</kp>
+      <kd>100.0</kd>
+      <mu1>1.0</mu1>
+      <mu2>1.0</mu2>
+      <fdir1>1 0 0</fdir1>
+      <maxVel>1.0</maxVel>
+      <minDepth>0.003</minDepth>
+      <implicitSpringDamper>1</implicitSpringDamper>
+    </gazebo>
   </xacro:macro>
 </robot>
