Commit message: created launch for multi-robots and added real caster wheels

File: urdf/bases/default_base.urdf.xacro (robot description, xacro)
@@ -1,10 +1,10 @@
 <?xml version="1.0"?>
 <robot xmlns:xacro="http://ros.org/wiki/xacro">
-  <xacro:macro name="default_base_macro" params="robot_namespace mass width height depth *origin">
+  <xacro:macro name="default_base_macro" params="robot_namespace mass width depth height *origin">
     <link name="${robot_namespace}/base_footprint"/>
     <joint name="${robot_namespace}/base_joint" type="fixed">
       <xacro:insert_block name="origin"/>
       <parent link="${robot_namespace}/base_footprint"/>
-      <child link="${robot_namespace}/base_link" />
+      <child link="${robot_namespace}/base_link"/>
     </joint>
     <link name="${robot_namespace}/base_link">
@@ -12,5 +12,5 @@
         <origin xyz="0 0 0" rpy="0 0 0"/>
         <geometry>
-          <box size="${width} ${height} ${depth}"/>
+          <box size="${width} ${depth} ${height}"/>
         </geometry>
         <material name="blue"/>
@@ -19,5 +19,5 @@
         <origin xyz="0 0 0" rpy="0 0 0"/>
         <geometry>
-          <box size="${width} ${height} ${depth}"/>
+          <box size="${width} ${depth} ${height}"/>
         </geometry>
       </collision>

File: urdf/controllers/differential_drive.gazebo.xacro (robot description, xacro)
@@ -4,5 +4,8 @@
     <gazebo>
       <plugin name="gazebo_ros_diff_drive" filename="libgazebo_ros_diff_drive.so">
-        <odometry_topic>${robot_namespace}/odometry/odom_unfiltered</odometry_topic>
+        <ros>
+          <remapping>odom:=odometry/odom_unfiltered</remapping>
+          <remapping>cmd_vel:=velocity_cmd</remapping>
+        </ros>
         <odometry_frame>${robot_namespace}/odom</odometry_frame>
         <update_rate>30</update_rate>
@@ -13,5 +16,4 @@
         <max_wheel_torque>${wheel_max_torque}</max_wheel_torque>
         <max_wheel_acceleration>${wheel_max_acceleration}</max_wheel_acceleration>
-        <command_topic>${robot_namespace}/velocity_cmd</command_topic>
         <publish_odom>true</publish_odom>
         <publish_odom_tf>true</publish_odom_tf>
@@ -19,9 +21,4 @@
         <robot_base_frame>${robot_namespace}/base_footprint</robot_base_frame>
       </plugin>
-      <plugin name="gazebo_ros_joint_state_publisher" filename="libgazebo_ros_joint_state_publisher.so">
-        <update_rate>30</update_rate>
-        <joint_name>${robot_namespace}/${right_wheel_prefix}_joint</joint_name>
-        <joint_name>${robot_namespace}/${left_wheel_prefix}_joint</joint_name>
-      </plugin>
     </gazebo>
   </xacro:macro>

File: urdf/inertias.urdf.xacro (robot description, xacro)
@@ -1,11 +1,4 @@
 <?xml version="1.0"?>
 <robot xmlns:xacro="http://ros.org/wiki/xacro">
-  <xacro:macro name="solid_sphere_inertia_macro" params="mass radius">
-    <inertia
-      ixx="${2 * radius * radius * mass / 5}"
-      iyy="${2 * radius * radius * mass / 5}"
-      izz="${2 * radius * radius * mass / 5}"
-      ixy="0" ixz="0" iyz="0"/>
-  </xacro:macro>
   <xacro:macro name="solid_cylinder_inertia_macro" params="mass radius height">
     <inertia
@@ -15,9 +8,9 @@
       ixy="0" ixz="0" iyz="0"/>
   </xacro:macro>
-  <xacro:macro name="solid_cuboid_inertia_macro" params="mass height depth width">
+  <xacro:macro name="solid_cuboid_inertia_macro" params="mass width depth height">
     <inertia
       ixx="${mass / 12 * (height * height + depth * depth)}"
-      iyy="${mass / 12 * (width * width + depth * depth)}"
-      izz="${mass / 12 * (width * width + height * height)}"
+      iyy="${mass / 12 * (width * width + height * height)}"
+      izz="${mass / 12 * (width * width + depth * depth)}"
       ixy="0" ixz="0" iyz="0"/>
   </xacro:macro>

File: urdf/palletron.xacro (robot description, xacro)
@@ -16,23 +16,33 @@
   <!-- Base parameters -->
   <xacro:property name="base_width" value="0.7"/>
-  <xacro:property name="base_height" value="0.7"/>
+  <xacro:property name="base_height" value="0.4"/>
   <xacro:property name="base_depth" value="0.7"/>
   <xacro:property name="base_mass" value="100"/>
   <!-- Drive wheels parameters -->
-  <xacro:property name="drive_wheel_mass" value="4.0"/>
-  <xacro:property name="drive_wheel_radius" value="0.13"/>
+  <xacro:property name="drive_wheel_mass" value="10.0"/>
+  <xacro:property name="drive_wheel_radius" value="0.12"/>
   <xacro:property name="drive_wheel_length" value="0.05"/>
   <xacro:property name="drive_wheel_separation" value="0.33"/>
-  <xacro:property name="drive_wheel_offset_z" value="-0.275"/>
+  <xacro:property name="drive_wheel_offset_z" value="-0.475"/>
   <xacro:property name="drive_wheel_max_acceleration" value="1.0"/>
-  <xacro:property name="drive_wheel_max_torque" value="6.0"/>
+  <xacro:property name="drive_wheel_max_torque" value="10.0"/>
   <xacro:property name="right_drive_wheel_prefix" value="right_wheel"/>
   <xacro:property name="left_drive_wheel_prefix" value="left_wheel"/>
   <!-- Caster wheels parameters -->
-  <xacro:property name="caster_radius" value="0.045"/>
-  <xacro:property name="caster_mass" value="0.005"/>
-  <xacro:property name="caster_offset_x" value="0.25"/>
-  <xacro:property name="caster_offset_y" value="0.25"/>
-  <xacro:property name="caster_offset_ground" value="0.005"/>
+  <xacro:property name="caster_wheel_mass" value="4.0"/>
+  <xacro:property name="caster_wheel_radius" value="0.045"/>
+  <xacro:property name="caster_wheel_length" value="0.05"/>
+  <xacro:property name="caster_wheel_offset_x" value="0.25"/>
+  <xacro:property name="caster_wheel_offset_y" value="0.25"/>
+  <xacro:property name="caster_wheel_offset_ground" value="0.005"/>
+  <xacro:property name="caster_mount_height" value ="0.0057"/>
+  <xacro:property name="caster_mount_offset_z" value="${-base_height / 2 - caster_mount_height}"/>
+  <xacro:property name="caster_fork_to_mount_offset_z" value="-0.02"/>
+  <xacro:property name="caster_wheel_to_fork_offset_z" value="-0.075"/>
+  <xacro:property name="front_right_caster_wheel_prefix" value="front_right_caster"/>
+  <xacro:property name="front_left_caster_wheel_prefix" value="front_left_caster"/>
+  <xacro:property name="rear_right_caster_wheel_prefix" value="rear_right_caster"/>
+  <xacro:property name="rear_left_caster_wheel_prefix" value="rear_left_caster"/>
+  <xacro:property name="base_footprint_offset_z" value="${caster_mount_offset_z + caster_fork_to_mount_offset_z + caster_wheel_to_fork_offset_z - (caster_wheel_radius / 2)}"/>
   <!-- Add default base -->
   <xacro:default_base_macro robot_namespace="${namespace}"
@@ -42,5 +52,5 @@
     depth="${base_depth}">
     <!-- Base footprint origin -->
-    <origin xyz="0 0 ${drive_wheel_radius - drive_wheel_offset_z}" rpy="0 0 0"/>
+    <origin xyz="0 0 ${-base_footprint_offset_z}" rpy="0 0 0"/>
   </xacro:default_base_macro>
   <!-- Add the differential drive plugin -->
@@ -60,5 +70,5 @@
     length="${drive_wheel_length}"
     parent="base_link">
-    <origin xyz="0 ${-drive_wheel_separation/2} ${drive_wheel_offset_z}" rpy="${-pi/2} 0 0"/>
+    <origin xyz="0 ${-drive_wheel_separation/2} ${-base_height / 2 - caster_mount_height + caster_fork_to_mount_offset_z + caster_wheel_to_fork_offset_z + (drive_wheel_radius - caster_wheel_radius)}" rpy="${-pi/2} 0 0"/>
   </xacro:drive_wheel_macro>
   <xacro:drive_wheel_macro robot_namespace="${namespace}"
@@ -68,34 +78,50 @@
     length="${drive_wheel_length}"
     parent="base_link">
-    <origin xyz="0 ${drive_wheel_separation/2} ${drive_wheel_offset_z}" rpy="${-pi/2} 0 0"/>
+    <origin xyz="0 ${drive_wheel_separation/2} ${-base_height / 2 - caster_mount_height + caster_fork_to_mount_offset_z + caster_wheel_to_fork_offset_z + (drive_wheel_radius - caster_wheel_radius)}" rpy="${-pi/2} 0 0"/>
   </xacro:drive_wheel_macro>
   <!-- Add four caster wheels -->
   <xacro:caster_wheel_macro robot_namespace="${namespace}"
-    prefix="front_right_caster"
-    mass="${caster_mass}"
-    radius="${caster_radius}"
+    prefix="${front_right_caster_wheel_prefix}"
+    wheel_mass="${caster_wheel_mass}"
+    wheel_radius="${caster_wheel_radius}"
+    wheel_length="${caster_wheel_length}"
+    mount_height="${caster_mount_height}"
+    fork_to_mount_offset_z="${caster_fork_to_mount_offset_z}"
+    wheel_to_fork_offset_z="${caster_wheel_to_fork_offset_z}"
     parent="base_link">
-    <origin xyz="-${caster_offset_x} ${caster_offset_y} ${drive_wheel_offset_z + caster_offset_ground - (drive_wheel_radius - caster_radius)}" rpy="0 0 0"/>
+    <origin xyz="-${caster_wheel_offset_x} ${caster_wheel_offset_y} ${-base_height / 2 - caster_mount_height / 2 + caster_wheel_offset_ground}" rpy="0 0 0"/>
   </xacro:caster_wheel_macro>
   <xacro:caster_wheel_macro robot_namespace="${namespace}"
-    prefix="front_left_caster"
-    mass="${caster_mass}"
-    radius="${caster_radius}"
+    prefix="${front_left_caster_wheel_prefix}"
+    wheel_mass="${caster_wheel_mass}"
+    wheel_radius="${caster_wheel_radius}"
+    wheel_length="${caster_wheel_length}"
+    mount_height="${caster_mount_height}"
+    fork_to_mount_offset_z="${caster_fork_to_mount_offset_z}"
+    wheel_to_fork_offset_z="${caster_wheel_to_fork_offset_z}"
     parent="base_link">
-    <origin xyz="${caster_offset_x} ${caster_offset_y} ${drive_wheel_offset_z + caster_offset_ground - (drive_wheel_radius - caster_radius)}" rpy="0 0 0"/>
+    <origin xyz="${caster_wheel_offset_x} ${caster_wheel_offset_y} ${-base_height / 2 - caster_mount_height / 2 + caster_wheel_offset_ground}" rpy="0 0 0"/>
   </xacro:caster_wheel_macro>
   <xacro:caster_wheel_macro robot_namespace="${namespace}"
-    prefix="rear_right_caster"
-    mass="${caster_mass}"
-    radius="${caster_radius}"
+    prefix="${rear_right_caster_wheel_prefix}"
+    wheel_mass="${caster_wheel_mass}"
+    wheel_radius="${caster_wheel_radius}"
+    wheel_length="${caster_wheel_length}"
+    mount_height="${caster_mount_height}"
+    fork_to_mount_offset_z="${caster_fork_to_mount_offset_z}"
+    wheel_to_fork_offset_z="${caster_wheel_to_fork_offset_z}"
     parent="base_link">
-    <origin xyz="-${caster_offset_x} -${caster_offset_y} ${drive_wheel_offset_z + caster_offset_ground - (drive_wheel_radius - caster_radius)}" rpy="0 0 0"/>
+    <origin xyz="-${caster_wheel_offset_x} -${caster_wheel_offset_y} ${-base_height/2 - caster_mount_height / 2 + caster_wheel_offset_ground}" rpy="0 0 0"/>
   </xacro:caster_wheel_macro>
   <xacro:caster_wheel_macro robot_namespace="${namespace}"
-    prefix="rear_left_caster"
-    mass="${caster_mass}"
-    radius="${caster_radius}"
+    prefix="${rear_left_caster_wheel_prefix}"
+    wheel_mass="${caster_wheel_mass}"
+    wheel_radius="${caster_wheel_radius}"
+    wheel_length="${caster_wheel_length}"
+    mount_height="${caster_mount_height}"
+    fork_to_mount_offset_z="${caster_fork_to_mount_offset_z}"
+    wheel_to_fork_offset_z="${caster_wheel_to_fork_offset_z}"
     parent="base_link">
-    <origin xyz="${caster_offset_x} -${caster_offset_y} ${drive_wheel_offset_z + caster_offset_ground - (drive_wheel_radius - caster_radius)}" rpy="0 0 0"/>
+    <origin xyz="${caster_wheel_offset_x} -${caster_wheel_offset_y} ${-base_height/2 - caster_mount_height / 2 + caster_wheel_offset_ground}" rpy="0 0 0"/>
   </xacro:caster_wheel_macro>
   <!-- Add a RPlidar -->

File: urdf/wheels/caster_wheel.urdf.xacro (robot description, xacro)
@@ -1,41 +1,100 @@
 <?xml version="1.0"?>
 <robot xmlns:xacro="http://ros.org/wiki/xacro">
-  <xacro:macro name="caster_wheel_macro" params="robot_namespace prefix mass radius parent *origin">
-    <link name="${robot_namespace}/${prefix}_link">
+  <xacro:macro name="caster_wheel_macro" params="robot_namespace prefix wheel_mass wheel_radius wheel_length mount_height fork_to_mount_offset_z wheel_to_fork_offset_z parent *origin">
+    <link name="${robot_namespace}/${prefix}_mount_link">
       <visual>
-        <origin xyz="0 0 0" rpy="0 0 0"/>
         <geometry>
-          <sphere radius="${radius}"/>
+          <box size="0.1145 0.1 ${mount_height}"/>
         </geometry>
-        <material name="grey"/>
+        <origin rpy="0 0 0" xyz="0 0 0"/>
+        <material name="black"/>
       </visual>
       <collision>
-        <origin xyz="0 0 0" rpy="0 0 0"/>
         <geometry>
-          <sphere radius="${radius}"/>
+          <box size="0.1145 0.1 ${mount_height}"/>
         </geometry>
+        <origin rpy="0 0 0" xyz="0 0 0"/>
       </collision>
       <inertial>
-        <origin xyz="0 0 0" rpy="0 0 0"/>
-        <mass value="${mass}"/>
-        <xacro:solid_sphere_inertia_macro mass="${mass}" radius="${radius}"/>
+        <origin rpy="0 0 0" xyz="0 0 0"/>
+        <mass value="0.25"/>
+        <inertia ixx="0.000209010208333" ixy="0" ixz="0" iyy="0.000273807083333" iyz="0" izz="0.000273807083333"/>
       </inertial>
     </link>
-    <joint name="${robot_namespace}/${prefix}_joint" type="fixed">
+    <joint name="${robot_namespace}/${prefix}_mount_joint" type="fixed">
+      <parent link="${robot_namespace}/${parent}"/>
+      <child link="${robot_namespace}/${prefix}_mount_link"/>
       <xacro:insert_block name="origin"/>
-      <parent link="${robot_namespace}/${parent}"/>
-      <child link="${robot_namespace}/${prefix}_link"/>
+    </joint>
+    <link name="${robot_namespace}/${prefix}_fork_link">
+      <visual>
+        <geometry>
+          <box size="0.02 0.02 0.02"/>
+        </geometry>
+        <origin rpy="0 0 0" xyz="0 0 0"/>
+        <material name="black"/>
+      </visual>
+      <collision>
+        <geometry>
+          <box size="0.02 0.02 0.02"/>
+        </geometry>
+        <origin rpy="0 0 0" xyz="0 0 0"/>
+      </collision>
+      <inertial>
+        <origin rpy="0 0 0" xyz="0 0 0"/>
+        <mass value="1.5"/>
+        <inertia ixx="0.0001" ixy="0" ixz="0" iyy="0.0001" iyz="0" izz="0.0001"/>
+      </inertial>
+    </link>
+    <joint name="${robot_namespace}/${prefix}_fork_joint" type="continuous">
+      <axis rpy="0 0 0" xyz="0 0 1"/>
+      <parent link="${robot_namespace}/${prefix}_mount_link"/>
+      <child link="${robot_namespace}/${prefix}_fork_link"/>
+      <origin xyz="0 0 ${fork_to_mount_offset_z}"/>
+      <dynamics damping="0.0" friction="0.15"/>
+    </joint>
+    <link name="${robot_namespace}/${prefix}_wheel_link">
+      <visual>
+        <geometry>
+          <cylinder length="${wheel_length}" radius="${wheel_radius}"/>
+        </geometry>
+        <origin rpy="${pi/2} 0 0" xyz="0 0 0"/>
+        <material name="orange"/>
+      </visual>
+      <collision>
+        <geometry>
+          <cylinder length="${wheel_length}" radius="${wheel_radius}"/>
+        </geometry>
+        <origin rpy="${pi/2} 0 0" xyz="0 0 0"/>
+      </collision>
+      <inertial>
+        <origin rpy="${pi/2} 0 0" xyz="0 0 0"/>
+        <mass value="${wheel_mass}"/>
+        <xacro:solid_cylinder_inertia_macro mass="${wheel_mass}" radius="${wheel_radius}" height="${wheel_length}"/>
+      </inertial>
+    </link>
+    <joint name="${robot_namespace}/${prefix}_wheel_joint" type="continuous">
+      <axis rpy="0 0 0" xyz="0 1 0"/>
+      <parent link="${robot_namespace}/${prefix}_fork_link"/>
+      <child link="${robot_namespace}/${prefix}_wheel_link"/>
+      <origin xyz="-0.037 0 ${wheel_to_fork_offset_z}"/>
+      <dynamics damping="0.0" friction="0.15"/>
     </joint>
     <!-- Gazebo extensions -->
-    <gazebo reference="${robot_namespace}/${prefix}_link">
+    <gazebo reference="${robot_namespace}/${prefix}_fork_link">
       <material>Gazebo/Grey</material>
+    </gazebo>
+    <gazebo reference="${robot_namespace}/${prefix}_mount_link">
+      <material>Gazebo/Grey</material>
+    </gazebo>
+    <gazebo reference="${robot_namespace}/${prefix}_wheel_link">
+      <material>Gazebo/Orange</material>
       <kp>1000000.0</kp>
-      <kd>100.0</kd>
-      <mu1>0.0</mu1>
-      <mu2>0.0</mu2>
+      <kd>10.0</kd>
+      <mu1>1.0</mu1>
+      <mu2>1.0</mu2>
       <fdir1>1 0 0</fdir1>
       <maxVel>1.0</maxVel>
-      <minDepth>0.0</minDepth>
-      <implicitSpringDamper>1</implicitSpringDamper>
+      <minDepth>0.00</minDepth>
     </gazebo>
   </xacro:macro>
