Commit message: changed the urdf to be similar to the Rhino

File: urdf/bases/base_without_mesh.urdf.xacro (robot description, xacro)
@@ -1,5 +1,5 @@
 <?xml version="1.0"?>
 <robot xmlns:xacro="http://ros.org/wiki/xacro">
-  <xacro:macro name="default_base_macro" params="robot_namespace mass width depth height *origin">
+  <xacro:macro name="base_without_mesh_macro" params="robot_namespace mass body_width body_length body_height *origin">
     <link name="${robot_namespace}/base_footprint"/>
     <joint name="${robot_namespace}/base_joint" type="fixed">
@@ -12,5 +12,5 @@
         <origin xyz="0 0 0" rpy="0 0 0"/>
         <geometry>
-          <box size="${width} ${depth} ${height}"/>
+          <box size="${body_width} ${body_length} ${body_height}"/>
         </geometry>
         <material name="blue"/>
@@ -19,5 +19,5 @@
         <origin xyz="0 0 0" rpy="0 0 0"/>
         <geometry>
-          <box size="${width} ${depth} ${height}"/>
+          <box size="${body_width} ${body_length} ${body_height}"/>
         </geometry>
       </collision>
@@ -25,21 +25,11 @@
         <origin xyz="0 0 0" rpy="0 0 0"/>
         <mass value="${mass}"/>
-        <xacro:solid_cuboid_inertia_macro mass="${mass}" height="${height}" depth="${depth}" width="${width}"/>
+        <xacro:cuboid_inertia_macro mass="${mass}" width="${body_width}" length="${body_length}" height="${body_height}"/>
       </inertial>
     </link>
-    <!-- Gazebo extensions -->
+    <!-- Gazebo elements -->
     <gazebo reference="${robot_namespace}/base_link">
       <material>Gazebo/Blue</material>
     </gazebo>
-    <gazebo reference="${robot_namespace}/base_footprint">
-      <kp>100000000.0</kp>
-      <kd>10.0</kd>
-      <mu1>0.1</mu1>
-      <mu2>0.1</mu2>
-      <fdir1>1 0 0</fdir1>
-      <maxVel>10.0</maxVel>
-      <minDepth>0.0005</minDepth>
-      <laserRetro>0</laserRetro>
-    </gazebo>
   </xacro:macro>
 </robot>

File: urdf/common_properties.urdf.xacro (robot description, xacro)
@@ -1,4 +1,5 @@
 <?xml version="1.0"?>
 <robot xmlns:xacro="http://wiki.ros.org/xacro">
+  <!-- Materials -->
   <material name="black">
       <color rgba="0.0 0.0 0.0 1.0"/>
@@ -34,3 +35,9 @@
     <color rgba="1.0 1.0 1.0 1.0"/>
   </material>
+  <!-- Math constants -->
+  <xacro:property name="rad0" value="0"/>
+  <xacro:property name="rad45" value="${45*pi/180}"/>
+  <xacro:property name="rad90" value="${90*pi/180}"/>
+  <xacro:property name="rad135" value="${135*pi/180}"/>
+  <xacro:property name="rad180" value="${180*pi/180}"/>
 </robot>

File: urdf/inertias.urdf.xacro (robot description, xacro)
@@ -1,16 +1,23 @@
 <?xml version="1.0"?>
 <robot xmlns:xacro="http://ros.org/wiki/xacro">
-  <xacro:macro name="solid_cylinder_inertia_macro" params="mass radius height">
+  <xacro:macro name="cuboid_inertia_macro" params="mass width length height">
     <inertia
-      ixx="${mass / 12 * (3 * radius * radius + height * height)}"
-      iyy="${mass / 12 * (3 * radius * radius + height * height)}"
+      ixx="${mass / 12 * (length * length + height * height)}"
+      iyy="${mass / 12 * (width * width + height * height)}"
+      izz="${mass / 12 * (width * width + length * length)}"
+      ixy="0" ixz="0" iyz="0"/>
+  </xacro:macro>
+  <xacro:macro name="cylinder_inertia_macro" params="mass radius length">
+    <inertia
+      ixx="${mass / 12 * (3 * radius * radius + length * length)}"
+      iyy="${mass / 12 * (3 * radius * radius + length * length)}"
       izz="${mass / 2 * (radius * radius)}"
       ixy="0" ixz="0" iyz="0"/>
   </xacro:macro>
-  <xacro:macro name="solid_cuboid_inertia_macro" params="mass width depth height">
+  <xacro:macro name="sphere_inertia_macro" params="mass radius">
     <inertia
-      ixx="${mass / 12 * (height * height + depth * depth)}"
-      iyy="${mass / 12 * (width * width + height * height)}"
-      izz="${mass / 12 * (width * width + depth * depth)}"
+      ixx="${2 * radius * radius * mass / 5}"
+      iyy="${2 * radius * radius * mass / 5}"
+      izz="${2 * radius * radius * mass / 5}"
       ixy="0" ixz="0" iyz="0"/>
   </xacro:macro>

File: urdf/palletron.xacro (robot description, xacro)
@@ -4,55 +4,49 @@
   <xacro:include filename="common_properties.urdf.xacro"/>
   <xacro:include filename="inertias.urdf.xacro"/>
-  <xacro:include filename="bases/default_base.urdf.xacro"/>
-  <xacro:include filename="controllers/differential_drive.gazebo.xacro"/>
+  <xacro:include filename="bases/base_without_mesh.urdf.xacro"/>
+  <xacro:include filename="plugins/differential_drive.gazebo.xacro"/>
   <xacro:include filename="wheels/drive_wheel.urdf.xacro"/>
-  <xacro:include filename="wheels/caster_wheel.urdf.xacro"/>
-  <xacro:include filename="sensors/rplidar.urdf.xacro"/>
-  <!-- Load optional properties files -->
-  <xacro:property name="namespace" value="$(arg namespace)" />
+  <xacro:include filename="wheels/dummy_caster_wheel.urdf.xacro"/>
+  <xacro:include filename="sensors/hokuyo.urdf.xacro"/>
+  <xacro:include filename="sensors/imu.urdf.xacro"/>
+  <!-- Load arguments -->
+  <xacro:property name="namespace" value="$(arg namespace)"/>
+  <!-- Load optional properties file -->
   <xacro:property name="optional_properties" value="$(arg optional_properties)"/>
   <xacro:property name="optionals" value="${xacro.load_yaml(optional_properties)}"/>
-  <!-- TODO: Update according to real properties -->
   <!-- Base parameters -->
-  <xacro:property name="base_width" value="0.7"/>
-  <xacro:property name="base_height" value="0.4"/>
-  <xacro:property name="base_depth" value="0.7"/>
-  <xacro:property name="base_mass" value="100"/>
+  <xacro:property name="mass" value="10.0"/>
+  <xacro:property name="base_width" value="0.6"/>
+  <xacro:property name="base_length" value="0.7"/>
+  <xacro:property name="base_height" value="0.7"/>
   <!-- Drive wheels parameters -->
-  <xacro:property name="drive_wheel_mass" value="10.0"/>
-  <xacro:property name="drive_wheel_radius" value="0.12"/>
-  <xacro:property name="drive_wheel_length" value="0.05"/>
-  <xacro:property name="drive_wheel_separation" value="0.33"/>
-  <xacro:property name="drive_wheel_offset_z" value="-0.475"/>
+  <xacro:property name="drive_wheel_mass" value="1.0"/>
+  <xacro:property name="drive_wheel_radius" value="0.045"/>
+  <xacro:property name="drive_wheel_width" value="0.03"/>
+  <xacro:property name="drive_wheel_offset_x" value="0.275"/>
+  <xacro:property name="drive_wheel_offset_z" value="${-base_height/2 - 0.08}"/>
+  <xacro:property name="drive_wheel_separation" value="0.45"/>
   <xacro:property name="drive_wheel_max_acceleration" value="1.0"/>
   <xacro:property name="drive_wheel_max_torque" value="10.0"/>
   <xacro:property name="right_drive_wheel_prefix" value="right_wheel"/>
   <xacro:property name="left_drive_wheel_prefix" value="left_wheel"/>
-  <!-- Caster wheels parameters -->
-  <xacro:property name="caster_wheel_mass" value="4.0"/>
-  <xacro:property name="caster_wheel_radius" value="0.045"/>
-  <xacro:property name="caster_wheel_length" value="0.05"/>
-  <xacro:property name="caster_wheel_offset_x" value="0.25"/>
-  <xacro:property name="caster_wheel_offset_y" value="0.25"/>
-  <xacro:property name="caster_wheel_offset_ground" value="0.005"/>
-  <xacro:property name="caster_mount_height" value ="0.0057"/>
-  <xacro:property name="caster_mount_offset_z" value="${-base_height / 2 - caster_mount_height}"/>
-  <xacro:property name="caster_fork_to_mount_offset_z" value="-0.02"/>
-  <xacro:property name="caster_wheel_to_fork_offset_z" value="-0.075"/>
-  <xacro:property name="front_right_caster_wheel_prefix" value="front_right_caster"/>
-  <xacro:property name="front_left_caster_wheel_prefix" value="front_left_caster"/>
-  <xacro:property name="rear_right_caster_wheel_prefix" value="rear_right_caster"/>
-  <xacro:property name="rear_left_caster_wheel_prefix" value="rear_left_caster"/>
-  <xacro:property name="base_footprint_offset_z" value="${caster_mount_offset_z + caster_fork_to_mount_offset_z + caster_wheel_to_fork_offset_z - (caster_wheel_radius / 2)}"/>
-  <!-- Add default base -->
-  <xacro:default_base_macro robot_namespace="${namespace}"
-    mass="${base_mass}"
-    width="${base_width}"
-    height="${base_height}"
-    depth="${base_depth}">
-    <!-- Base footprint origin -->
-    <origin xyz="0 0 ${-base_footprint_offset_z}" rpy="0 0 0"/>
-  </xacro:default_base_macro>
-  <!-- Add the differential drive plugin -->
+  <!-- Dummy caster wheels parameters -->
+  <xacro:property name="dummy_caster_wheel_mass" value="0.0001"/>
+  <xacro:property name="dummy_caster_wheel_radius" value="0.035"/>
+  <xacro:property name="dummy_caster_wheel_width" value="0.03"/>
+  <xacro:property name="dummy_caster_wheel_offset_x" value="1.00"/>
+  <xacro:property name="dummy_caster_wheel_offset_y" value="0.0"/>
+  <xacro:property name="dummy_caster_wheel_offset_ground" value="0.025"/>
+  <xacro:property name="dummy_caster_wheel_prefix" value="front_caster_wheel"/>
+  <!-- Base without mesh -->
+  <xacro:base_without_mesh_macro robot_namespace="${namespace}"
+    mass="${mass}"
+    body_width="${base_width}"
+    body_length="${base_length}"
+    body_height="${base_height}">
+    <!-- Base link origin -->
+    <origin xyz="0 0 ${drive_wheel_radius - drive_wheel_offset_z}" rpy="0 0 0"/>
+  </xacro:base_without_mesh_macro>
+  <!-- Differential drive plugin -->
   <xacro:differential_drive_macro robot_namespace="${namespace}"
     right_wheel_prefix="${right_drive_wheel_prefix}"
@@ -63,75 +57,51 @@
     wheel_max_acceleration="${drive_wheel_max_acceleration}">
   </xacro:differential_drive_macro>
-  <!-- Add two drive wheels -->
+  <!-- Right drive wheel -->
   <xacro:drive_wheel_macro robot_namespace="${namespace}"
+    parent="base_link"
     prefix="${right_drive_wheel_prefix}"
     mass="${drive_wheel_mass}"
     radius="${drive_wheel_radius}"
-    length="${drive_wheel_length}"
-    parent="base_link">
-    <origin xyz="0 ${-drive_wheel_separation/2} ${-base_height / 2 - caster_mount_height + caster_fork_to_mount_offset_z + caster_wheel_to_fork_offset_z + (drive_wheel_radius - caster_wheel_radius)}" rpy="${-pi/2} 0 0"/>
+    length="${drive_wheel_width}"
+    xyz="${drive_wheel_offset_x} ${-drive_wheel_separation/2} ${drive_wheel_offset_z}">
   </xacro:drive_wheel_macro>
+  <!-- Left drive wheel -->
   <xacro:drive_wheel_macro robot_namespace="${namespace}"
+    parent="base_link"
     prefix="${left_drive_wheel_prefix}"
     mass="${drive_wheel_mass}"
     radius="${drive_wheel_radius}"
-    length="${drive_wheel_length}"
-    parent="base_link">
-    <origin xyz="0 ${drive_wheel_separation/2} ${-base_height / 2 - caster_mount_height + caster_fork_to_mount_offset_z + caster_wheel_to_fork_offset_z + (drive_wheel_radius - caster_wheel_radius)}" rpy="${-pi/2} 0 0"/>
+    length="${drive_wheel_width}"
+    xyz="${drive_wheel_offset_x} ${drive_wheel_separation/2} ${drive_wheel_offset_z}">
   </xacro:drive_wheel_macro>
-  <!-- Add four caster wheels -->
-  <xacro:caster_wheel_macro robot_namespace="${namespace}"
-    prefix="${front_right_caster_wheel_prefix}"
-    wheel_mass="${caster_wheel_mass}"
-    wheel_radius="${caster_wheel_radius}"
-    wheel_length="${caster_wheel_length}"
-    mount_height="${caster_mount_height}"
-    fork_to_mount_offset_z="${caster_fork_to_mount_offset_z}"
-    wheel_to_fork_offset_z="${caster_wheel_to_fork_offset_z}"
-    parent="base_link">
-    <origin xyz="-${caster_wheel_offset_x} ${caster_wheel_offset_y} ${-base_height / 2 - caster_mount_height / 2 + caster_wheel_offset_ground}" rpy="0 0 0"/>
-  </xacro:caster_wheel_macro>
-  <xacro:caster_wheel_macro robot_namespace="${namespace}"
-    prefix="${front_left_caster_wheel_prefix}"
-    wheel_mass="${caster_wheel_mass}"
-    wheel_radius="${caster_wheel_radius}"
-    wheel_length="${caster_wheel_length}"
-    mount_height="${caster_mount_height}"
-    fork_to_mount_offset_z="${caster_fork_to_mount_offset_z}"
-    wheel_to_fork_offset_z="${caster_wheel_to_fork_offset_z}"
-    parent="base_link">
-    <origin xyz="${caster_wheel_offset_x} ${caster_wheel_offset_y} ${-base_height / 2 - caster_mount_height / 2 + caster_wheel_offset_ground}" rpy="0 0 0"/>
-  </xacro:caster_wheel_macro>
-  <xacro:caster_wheel_macro robot_namespace="${namespace}"
-    prefix="${rear_right_caster_wheel_prefix}"
-    wheel_mass="${caster_wheel_mass}"
-    wheel_radius="${caster_wheel_radius}"
-    wheel_length="${caster_wheel_length}"
-    mount_height="${caster_mount_height}"
-    fork_to_mount_offset_z="${caster_fork_to_mount_offset_z}"
-    wheel_to_fork_offset_z="${caster_wheel_to_fork_offset_z}"
-    parent="base_link">
-    <origin xyz="-${caster_wheel_offset_x} -${caster_wheel_offset_y} ${-base_height/2 - caster_mount_height / 2 + caster_wheel_offset_ground}" rpy="0 0 0"/>
-  </xacro:caster_wheel_macro>
-  <xacro:caster_wheel_macro robot_namespace="${namespace}"
-    prefix="${rear_left_caster_wheel_prefix}"
-    wheel_mass="${caster_wheel_mass}"
-    wheel_radius="${caster_wheel_radius}"
-    wheel_length="${caster_wheel_length}"
-    mount_height="${caster_mount_height}"
-    fork_to_mount_offset_z="${caster_fork_to_mount_offset_z}"
-    wheel_to_fork_offset_z="${caster_wheel_to_fork_offset_z}"
-    parent="base_link">
-    <origin xyz="${caster_wheel_offset_x} -${caster_wheel_offset_y} ${-base_height/2 - caster_mount_height / 2 + caster_wheel_offset_ground}" rpy="0 0 0"/>
-  </xacro:caster_wheel_macro>
-  <!-- Add a RPlidar -->
-  <xacro:rplidar_macro robot_namespace="${namespace}"
-    x="0"
-    y="0"
-    z="${base_height / 2}"
-    roll="0"
-    pitch="0"
-    yaw="0"
-    parent="base_link">
-  </xacro:rplidar_macro>
+  <!-- Dummy caster wheel -->
+  <xacro:dummy_caster_wheel_macro robot_namespace="${namespace}"
+    parent="base_link"
+    prefix="${dummy_caster_wheel_prefix}"
+    xyz="-${dummy_caster_wheel_offset_x} ${dummy_caster_wheel_offset_y} ${drive_wheel_offset_z + dummy_caster_wheel_offset_ground - (drive_wheel_radius - dummy_caster_wheel_radius)}">
+  </xacro:dummy_caster_wheel_macro>
+  <!-- Right laser ranger scanner -->
+  <xacro:hokuyo_macro robot_namespace="${namespace}"
+    parent="base_link"
+    prefix="right">
+    <origin xyz="${base_width/2 + 0.025} -${base_length/2 + 0.025} ${-base_height/2}" rpy="${rad180} 0 ${-rad45}"/>
+  </xacro:hokuyo_macro>
+  <!-- Left laser ranger scanner -->
+  <xacro:hokuyo_macro robot_namespace="${namespace}"
+    parent="base_link"
+    prefix="left">
+    <origin xyz="-${base_width/2 + 0.025} ${base_length/2 + 0.025} ${-base_height/2}" rpy="${rad180} 0 ${rad135}"/>
+  </xacro:hokuyo_macro>
+  <!-- IMU 1 -->
+  <xacro:imu_macro robot_namespace="${namespace}"
+    parent="base_link"
+    suffix="1">
+    <origin xyz="0 0 0" rpy="0 0 0"/>
+  </xacro:imu_macro>
+  <!-- IMU 2 -->
+  <xacro:imu_macro robot_namespace="${namespace}"
+    parent="base_link"
+    suffix="2">
+    <origin xyz="0 0 0" rpy="0 0 0"/>
+  </xacro:imu_macro>
 </robot>

File: urdf/plugins/differential_drive.gazebo.xacro (robot description, xacro)
@@ -5,9 +5,9 @@
       <plugin name="gazebo_ros_diff_drive" filename="libgazebo_ros_diff_drive.so">
         <ros>
-          <remapping>odom:=odometry/odom_unfiltered</remapping>
+          <remapping>odom:=odometry/unfiltered</remapping>
           <remapping>cmd_vel:=velocity_cmd</remapping>
         </ros>
         <odometry_frame>${robot_namespace}/odom</odometry_frame>
-        <update_rate>30</update_rate>
+        <update_rate>100</update_rate>
         <left_joint>${robot_namespace}/${left_wheel_prefix}_joint</left_joint>
         <right_joint>${robot_namespace}/${right_wheel_prefix}_joint</right_joint>

File: urdf/wheels/caster_wheel.urdf.xacro (robot description, xacro)
@@ -1,100 +1,94 @@
 <?xml version="1.0"?>
 <robot xmlns:xacro="http://ros.org/wiki/xacro">
-  <xacro:macro name="caster_wheel_macro" params="robot_namespace prefix wheel_mass wheel_radius wheel_length mount_height fork_to_mount_offset_z wheel_to_fork_offset_z parent *origin">
-    <link name="${robot_namespace}/${prefix}_mount_link">
+  <xacro:macro name="caster_wheel_macro" params="robot_namespace parent prefix wheel_mass wheel_radius wheel_width plate_height plate_to_swivel_offset_z swivel_to_wheel_offset_z xyz">
+    <!-- Plate -->
+    <link name="${robot_namespace}/${prefix}_plate_link">
       <visual>
+        <origin rpy="0 0 0" xyz="0 0 0"/>
         <geometry>
-          <box size="0.1145 0.1 ${mount_height}"/>
+          <box size="0.1145 0.1 ${plate_height}"/>
         </geometry>
-        <origin rpy="0 0 0" xyz="0 0 0"/>
-        <material name="black"/>
+        <material name="grey"/>
       </visual>
       <collision>
+        <origin rpy="0 0 0" xyz="0 0 0"/>
         <geometry>
-          <box size="0.1145 0.1 ${mount_height}"/>
+          <box size="0.1145 0.1 ${plate_height}"/>
         </geometry>
-        <origin rpy="0 0 0" xyz="0 0 0"/>
       </collision>
       <inertial>
+        <mass value="25.0"/>
         <origin rpy="0 0 0" xyz="0 0 0"/>
-        <mass value="0.25"/>
-        <inertia ixx="0.000209010208333" ixy="0" ixz="0" iyy="0.000273807083333" iyz="0" izz="0.000273807083333"/>
+        <xacro:cuboid_inertia_macro mass="25.0" width="0.1145" depth="0.1" height="${plate_height}"/>
       </inertial>
     </link>
-    <joint name="${robot_namespace}/${prefix}_mount_joint" type="fixed">
+    <joint name="${robot_namespace}/${prefix}_plate_joint" type="fixed">
+      <origin xyz="${xyz}" rpy="0 0 0"/>
       <parent link="${robot_namespace}/${parent}"/>
-      <child link="${robot_namespace}/${prefix}_mount_link"/>
-      <xacro:insert_block name="origin"/>
+      <child link="${robot_namespace}/${prefix}_plate_link"/>
     </joint>
-    <link name="${robot_namespace}/${prefix}_fork_link">
+    <!-- Swivel -->
+    <link name="${robot_namespace}/${prefix}_swivel_link">
       <visual>
+        <origin rpy="0 0 0" xyz="0 0 0"/>
         <geometry>
           <box size="0.02 0.02 0.02"/>
         </geometry>
-        <origin rpy="0 0 0" xyz="0 0 0"/>
-        <material name="black"/>
+        <material name="grey"/>
       </visual>
       <collision>
+        <origin rpy="0 0 0" xyz="0 0 0"/>
         <geometry>
           <box size="0.02 0.02 0.02"/>
         </geometry>
-        <origin rpy="0 0 0" xyz="0 0 0"/>
       </collision>
       <inertial>
+        <mass value="1.5"/>
         <origin rpy="0 0 0" xyz="0 0 0"/>
-        <mass value="1.5"/>
-        <inertia ixx="0.0001" ixy="0" ixz="0" iyy="0.0001" iyz="0" izz="0.0001"/>
+        <xacro:cuboid_inertia_macro mass="1.5" width="0.02" depth="0.02" height="0.02"/>
       </inertial>
     </link>
-    <joint name="${robot_namespace}/${prefix}_fork_joint" type="continuous">
-      <axis rpy="0 0 0" xyz="0 0 1"/>
-      <parent link="${robot_namespace}/${prefix}_mount_link"/>
-      <child link="${robot_namespace}/${prefix}_fork_link"/>
-      <origin xyz="0 0 ${fork_to_mount_offset_z}"/>
-      <dynamics damping="0.0" friction="0.15"/>
+    <joint name="${robot_namespace}/${prefix}_swivel_joint" type="continuous">
+      <origin xyz="0 0 ${plate_to_swivel_offset_z}"/>
+      <parent link="${robot_namespace}/${prefix}_plate_link"/>
+      <child link="${robot_namespace}/${prefix}_swivel_link"/>
+      <axis xyz="0 0 1"/>
     </joint>
+    <!-- Wheel -->
     <link name="${robot_namespace}/${prefix}_wheel_link">
       <visual>
+        <origin rpy="${rad90} 0 0" xyz="0 0 0"/>
         <geometry>
-          <cylinder length="${wheel_length}" radius="${wheel_radius}"/>
+          <cylinder length="${wheel_width}" radius="${wheel_radius}"/>
         </geometry>
-        <origin rpy="${pi/2} 0 0" xyz="0 0 0"/>
         <material name="orange"/>
       </visual>
       <collision>
+        <origin rpy="${rad90} 0 0" xyz="0 0 0"/>
         <geometry>
-          <cylinder length="${wheel_length}" radius="${wheel_radius}"/>
+          <cylinder length="${wheel_width}" radius="${wheel_radius}"/>
         </geometry>
-        <origin rpy="${pi/2} 0 0" xyz="0 0 0"/>
       </collision>
       <inertial>
-        <origin rpy="${pi/2} 0 0" xyz="0 0 0"/>
         <mass value="${wheel_mass}"/>
-        <xacro:solid_cylinder_inertia_macro mass="${wheel_mass}" radius="${wheel_radius}" height="${wheel_length}"/>
+        <origin rpy="${rad90} 0 0" xyz="0 0 0"/>
+        <xacro:cylinder_inertia_macro mass="${wheel_mass}" radius="${wheel_radius}" height="${wheel_width}"/>
       </inertial>
     </link>
     <joint name="${robot_namespace}/${prefix}_wheel_joint" type="continuous">
+      <origin xyz="-0.037 0 ${swivel_to_wheel_offset_z}"/>
+      <parent link="${robot_namespace}/${prefix}_swivel_link"/>
+      <child link="${robot_namespace}/${prefix}_wheel_link"/>
       <axis rpy="0 0 0" xyz="0 1 0"/>
-      <parent link="${robot_namespace}/${prefix}_fork_link"/>
-      <child link="${robot_namespace}/${prefix}_wheel_link"/>
-      <origin xyz="-0.037 0 ${wheel_to_fork_offset_z}"/>
-      <dynamics damping="0.0" friction="0.15"/>
     </joint>
-    <!-- Gazebo extensions -->
-    <gazebo reference="${robot_namespace}/${prefix}_fork_link">
+    <!-- Gazebo elements -->
+    <gazebo reference="${robot_namespace}/${prefix}_plate_link">
       <material>Gazebo/Grey</material>
     </gazebo>
-    <gazebo reference="${robot_namespace}/${prefix}_mount_link">
+    <gazebo reference="${robot_namespace}/${prefix}_swivel_link">
       <material>Gazebo/Grey</material>
     </gazebo>
     <gazebo reference="${robot_namespace}/${prefix}_wheel_link">
       <material>Gazebo/Orange</material>
-      <kp>1000000.0</kp>
-      <kd>10.0</kd>
-      <mu1>1.0</mu1>
-      <mu2>1.0</mu2>
-      <fdir1>1 0 0</fdir1>
-      <maxVel>1.0</maxVel>
-      <minDepth>0.00</minDepth>
     </gazebo>
   </xacro:macro>
