Commit message: changed the urdf to be similar to the Rhino

File: urdf/wheels/dummy_caster_wheel.urdf.xacro (robot description, xacro)
@@ -1,10 +1,10 @@
 <?xml version="1.0"?>
 <robot xmlns:xacro="http://ros.org/wiki/xacro">
-  <xacro:macro name="drive_wheel_macro" params="robot_namespace parent prefix mass radius length xyz">
+  <xacro:macro name="dummy_caster_wheel_macro" params="robot_namespace parent prefix xyz">
     <link name="${robot_namespace}/${prefix}_link">
       <visual>
         <origin xyz="0 0 0" rpy="0 0 0"/>
         <geometry>
-          <cylinder radius="${radius}" length="${length}"/>
+          <sphere radius="${radius}"/>
         </geometry>
         <material name="flat_black"/>
@@ -13,28 +13,30 @@
         <origin xyz="0 0 0" rpy="0 0 0"/>
         <geometry>
-          <cylinder radius="${radius}" length="${length}"/>
+          <sphere radius="${radius}"/>
         </geometry>
       </collision>
       <inertial>
         <origin xyz="0 0 0" rpy="0 0 0"/>
-        <mass value="${mass}"/>
-        <xacro:cylinder_inertia_macro mass="${mass}" radius="${radius}" length="${length}"/>
+        <mass value="0.01"/>
+        <inertia ixx="0.0001" ixy="0" ixz="0"
+                 iyy="0.0001" iyz="0"
+                 izz="0.0001"/>
       </inertial>
     </link>
-    <joint name="${robot_namespace}/${prefix}_joint" type="continuous">
-      <origin xyz="${xyz}" rpy="${-rad90} 0 0"/>
+    <joint name="${robot_namespace}/${prefix}_joint" type="fixed">
+      <origin xyz="${xyz}" rpy="0 0 0"/>
       <parent link="${robot_namespace}/${parent}"/>
       <child link="${robot_namespace}/${prefix}_link"/>
-      <axis xyz="0 0 1"/>
     </joint>
     <!-- Gazebo elements -->
     <gazebo reference="${robot_namespace}/${prefix}_link">
       <material>Gazebo/FlatBlack</material>
-      <kp>5000000.0</kp>
+      <kp>1000000.0</kp>
       <kd>100.0</kd>
-      <mu1>1.0</mu1>
-      <mu2>1.0</mu2>
+      <mu1>0.0</mu1>
+      <mu2>0.0</mu2>
+      <fdir1>1 0 0</fdir1>
       <maxVel>1.0</maxVel>
-      <minDepth>0.002</minDepth>
+      <minDepth>0.0</minDepth>
     </gazebo>
   </xacro:macro>
