Commit message: reorganized urdf folder (again) and fixed rplidar sensor

File: urdf/common_properties.urdf.xacro (robot description, xacro)
@@ -1,7 +1,9 @@
 <?xml version="1.0"?>
 <robot xmlns:xacro="http://wiki.ros.org/xacro">
-  <!-- Materials -->
   <material name="black">
       <color rgba="0.0 0.0 0.0 1.0"/>
+  </material>
+  <material name="flat_black">
+    <color rgba="0.1 0.1 0.1 1.0"/>
   </material>
   <material name="dark">
@@ -32,13 +34,3 @@
     <color rgba="1.0 1.0 1.0 1.0"/>
   </material>
-  <!-- Inertia -->
-  <xacro:macro name="sphere_inertia" params="m r">
-    <inertia ixx="${(2*r*r*m)/5}" ixy="0" ixz="0" iyy="${(2*r*r*m)/5}" iyz="0" izz="${(2*r*r*m)/5}"/>
-  </xacro:macro>
-  <xacro:macro name="cylinder_inertia" params="m r h">
-    <inertia ixx="${m*(3*r*r+h*h)/12}" ixy="0" ixz="0" iyy="${m*(3*r*r+h*h)/12}" iyz="0" izz="${m*r*r/2}"/>
-  </xacro:macro>
-  <xacro:macro name="box_inertia" params="m h d w">
-    <inertia ixx="${(m*(h*h+d*d))/12}" ixy="0" ixz="0" iyy="${(m*(w*w+d*d))/12}" iyz="0" izz="${(m*(w*w+h*h))/12}"/>
-  </xacro:macro>
 </robot>

File: urdf/wheels/caster_wheel.gazebo.xacro (robot description, xacro)
@@ -1,9 +1,7 @@
 <?xml version="1.0"?>
 <robot xmlns:xacro="http://ros.org/wiki/xacro">
-  <xacro:macro name="caster_wheel_gazebo" params="name">
-    <gazebo reference="${name}_link">
-      <!-- Material -->
+  <xacro:macro name="caster_wheel_gazebo_macro">
+    <gazebo reference="${prefix}_link">
       <material>Gazebo/Grey</material>
-      <!-- Contact model -->
       <kp>1000000.0</kp>
       <kd>100.0</kd>

File: urdf/wheels/caster_wheel.urdf.xacro (robot description, xacro)
@@ -1,8 +1,7 @@
 <?xml version="1.0"?>
 <robot xmlns:xacro="http://ros.org/wiki/xacro">
-  <!-- Includes -->
   <xacro:include filename="caster_wheel.gazebo.xacro"/>
-  <xacro:macro name="caster_wheel" params="name radius mass x_offset y_offset z_offset parent">
-    <link name="${name}_link">
+  <xacro:macro name="caster_wheel_macro" params="prefix mass radius parent *origin">
+    <link name="${prefix}_link">
       <visual>
         <origin xyz="0 0 0" rpy="0 0 0"/>
@@ -17,22 +16,18 @@
           <sphere radius="${radius}"/>
         </geometry>
-        <material name="orange"/>
       </collision>
       <inertial>
         <origin xyz="0 0 0" rpy="0 0 0"/>
-        <mass value="0.005"/>
-        <inertia ixx="0.001" ixy="0" ixz="0"
-                 iyy="0.001" iyz="0"
-                 izz="0.001"/>
-        <inertia />
+        <mass value="${mass}"/>
+        <xacro:solid_sphere_inertia_macro mass="${mass}" radius="${radius}"/>
       </inertial>
     </link>
-    <joint name="${name}_joint" type="fixed">
-      <origin xyz="${x_offset} ${y_offset} ${z_offset}" rpy="0 0 0"/>
+    <joint name="${prefix}_joint" type="fixed">
+      <xacro:insert_block name="origin"/>
       <parent link="${parent}"/>
-      <child link="${name}_link"/>
+      <child link="${prefix}_link"/>
     </joint>
-    <!-- Gazebo extensions -->
-    <xacro:caster_wheel_gazebo name="${name}"/>
+    <!-- Include Gazebo extensions -->
+    <xacro:caster_wheel_gazebo_macro/>
   </xacro:macro>
 </robot>

File: urdf/wheels/drive_wheel.gazebo.xacro (robot description, xacro)
@@ -1,9 +1,7 @@
 <?xml version="1.0"?>
 <robot xmlns:xacro="http://ros.org/wiki/xacro">
-  <xacro:macro name="drive_wheel_gazebo" params="name">
-    <gazebo reference="${name}_link">
-      <!-- Material -->
+  <xacro:macro name="drive_wheel_gazebo_macro">
+    <gazebo reference="${prefix}_link">
       <material>Gazebo/Black</material>
-      <!-- Contact model -->
       <kp>100000.0</kp>
       <kd>100.0</kd>

File: urdf/wheels/drive_wheel.urdf.xacro (robot description, xacro)
@@ -1,12 +1,11 @@
 <?xml version="1.0"?>
 <robot xmlns:xacro="http://ros.org/wiki/xacro">
-  <!-- Includes -->
   <xacro:include filename="drive_wheel.gazebo.xacro"/>
-  <xacro:macro name="drive_wheel" params="name radius mass z_offset width separation reflect parent">
-    <link name="${name}_link">
+  <xacro:macro name="drive_wheel_macro" params="prefix mass radius length parent *origin">
+    <link name="${prefix}_link">
       <visual>
         <origin xyz="0 0 0" rpy="0 0 0"/>
         <geometry>
-          <cylinder radius="${radius}" length="${width}"/>
+          <cylinder radius="${radius}" length="${length}"/>
         </geometry>
         <material name="black"/>
@@ -15,22 +14,21 @@
         <origin xyz="0 0 0" rpy="0 0 0"/>
         <geometry>
-          <cylinder radius="${radius}" length="${width}"/>
+          <cylinder radius="${radius}" length="${length}"/>
         </geometry>
-        <material name="orange"/>
       </collision>
       <inertial>
-        <origin xyz="0 0 ${-0.00207 * reflect}" rpy="0 0 0"/>
+        <origin xyz="0 0 0" rpy="0 0 0"/>
         <mass value="${mass}"/>
-        <xacro:cylinder_inertia m="${mass}" r="${radius}" h="${width}"/>
+        <xacro:solid_cylinder_inertia_macro mass="${mass}" radius="${radius}" height="${length}"/>
       </inertial>
     </link>
-    <joint name="${name}_joint" type="continuous">
-      <origin xyz="0 ${-separation / 2 * reflect} ${z_offset}" rpy="${-pi/2} 0 0"/>
+    <joint name="${prefix}_joint" type="continuous">
+      <xacro:insert_block name="origin"/>
       <parent link="${parent}"/>
-      <child link="${name}_link"/>
+      <child link="${prefix}_link"/>
       <axis xyz="0 0 1"/>
     </joint>
-    <!-- Gazebo extensions -->
-    <xacro:drive_wheel_gazebo name="${name}"/>
+    <!-- Include Gazebo extensions -->
+    <xacro:drive_wheel_gazebo_macro/>
   </xacro:macro>
 </robot>

Commit message: added ground truth plugin, removed Rviz files and fixed relationship between frames

File: urdf/common_properties.urdf.xacro (robot description, xacro)
@@ -37,7 +37,10 @@
   <!-- Math constants -->
   <xacro:property name="rad0" value="0"/>
+  <xacro:property name="rad30" value="${30*pi/180}" />
   <xacro:property name="rad45" value="${45*pi/180}"/>
   <xacro:property name="rad90" value="${90*pi/180}"/>
   <xacro:property name="rad135" value="${135*pi/180}"/>
+  <xacro:property name="rad150" value="${150*pi/180}" />
   <xacro:property name="rad180" value="${180*pi/180}"/>
+  <xacro:property name="rad210" value="${210*pi/180}" />
 </robot>

File: urdf/palletron.xacro (robot description, xacro)
@@ -4,10 +4,11 @@
   <xacro:include filename="common_properties.urdf.xacro"/>
   <xacro:include filename="inertias.urdf.xacro"/>
-  <xacro:include filename="bases/base_without_mesh.urdf.xacro"/>
-  <xacro:include filename="plugins/differential_drive.gazebo.xacro"/>
+  <xacro:include filename="chassis/chassis_without_mesh.urdf.xacro"/>
+  <xacro:include filename="plugins/differential_drive_plugin.gazebo.xacro"/>
+  <xacro:include filename="plugins/p3d_plugin.gazebo.xacro"/>
+  <xacro:include filename="sensors/hokuyo.urdf.xacro"/>
+  <xacro:include filename="sensors/imu.urdf.xacro"/>
   <xacro:include filename="wheels/drive_wheel.urdf.xacro"/>
   <xacro:include filename="wheels/dummy_caster_wheel.urdf.xacro"/>
-  <xacro:include filename="sensors/hokuyo.urdf.xacro"/>
-  <xacro:include filename="sensors/imu.urdf.xacro"/>
   <!-- Load arguments -->
   <xacro:property name="namespace" value="$(arg namespace)"/>
@@ -15,15 +16,15 @@
   <xacro:property name="optional_properties" value="$(arg optional_properties)"/>
   <xacro:property name="optionals" value="${xacro.load_yaml(optional_properties)}"/>
-  <!-- Base parameters -->
+  <!-- Chassis parameters -->
   <xacro:property name="mass" value="10.0"/>
-  <xacro:property name="base_width" value="0.6"/>
-  <xacro:property name="base_length" value="0.7"/>
-  <xacro:property name="base_height" value="0.7"/>
+  <xacro:property name="chassis_width" value="0.6"/>
+  <xacro:property name="chassis_length" value="0.7"/>
+  <xacro:property name="chassis_height" value="0.7"/>
+  <xacro:property name="chassis_offset_x" value="-0.275"/>
+  <xacro:property name="chassis_offset_z" value="0.45"/>
   <!-- Drive wheels parameters -->
   <xacro:property name="drive_wheel_mass" value="1.0"/>
   <xacro:property name="drive_wheel_radius" value="0.045"/>
   <xacro:property name="drive_wheel_width" value="0.03"/>
-  <xacro:property name="drive_wheel_offset_x" value="0.275"/>
-  <xacro:property name="drive_wheel_offset_z" value="${-base_height/2 - 0.08}"/>
   <xacro:property name="drive_wheel_separation" value="0.45"/>
   <xacro:property name="drive_wheel_max_acceleration" value="1.0"/>
@@ -32,29 +33,29 @@
   <xacro:property name="left_drive_wheel_prefix" value="left_wheel"/>
   <!-- Dummy caster wheels parameters -->
-  <xacro:property name="dummy_caster_wheel_mass" value="0.0001"/>
-  <xacro:property name="dummy_caster_wheel_radius" value="0.035"/>
-  <xacro:property name="dummy_caster_wheel_width" value="0.03"/>
-  <xacro:property name="dummy_caster_wheel_offset_x" value="1.00"/>
+  <xacro:property name="dummy_caster_wheel_radius" value="0.045"/>
+  <xacro:property name="dummy_caster_wheel_offset_x" value="-1.425"/>
   <xacro:property name="dummy_caster_wheel_offset_y" value="0.0"/>
-  <xacro:property name="dummy_caster_wheel_offset_ground" value="0.025"/>
+  <xacro:property name="dummy_caster_wheel_offset_ground" value="0.00125"/>
   <xacro:property name="dummy_caster_wheel_prefix" value="front_caster_wheel"/>
-  <!-- Base without mesh -->
-  <xacro:base_without_mesh_macro robot_namespace="${namespace}"
+  <!-- Chassis without mesh -->
+  <xacro:chassis_without_mesh_macro robot_namespace="${namespace}"
     mass="${mass}"
-    body_width="${base_width}"
-    body_length="${base_length}"
-    body_height="${base_height}">
-    <!-- Base link origin -->
-    <origin xyz="0 0 ${drive_wheel_radius - drive_wheel_offset_z}" rpy="0 0 0"/>
-  </xacro:base_without_mesh_macro>
+    chassis_width="${chassis_width}"
+    chassis_length="${chassis_length}"
+    chassis_height="${chassis_height}">
+    <!-- Base footprint origin (from base link) -->
+    <origin xyz="0 0 ${-drive_wheel_radius}" rpy="0 0 0"/>
+    <!-- Chassis origin (from base link) -->
+    <origin xyz="${chassis_offset_x} 0 ${chassis_offset_z}" rpy="0 0 0"/>
+  </xacro:chassis_without_mesh_macro>
   <!-- Differential drive plugin -->
-  <xacro:differential_drive_macro robot_namespace="${namespace}"
+  <xacro:differential_drive_plugin_macro robot_namespace="${namespace}"
     right_wheel_prefix="${right_drive_wheel_prefix}"
     left_wheel_prefix="${left_drive_wheel_prefix}"
     wheel_separation="${drive_wheel_separation}"
-    wheel_diameter="${drive_wheel_radius * 2}"
+    wheel_diameter="${drive_wheel_radius*2}"
     wheel_max_torque="${drive_wheel_max_torque}"
     wheel_max_acceleration="${drive_wheel_max_acceleration}">
-  </xacro:differential_drive_macro>
+  </xacro:differential_drive_plugin_macro>
   <!-- Right drive wheel -->
   <xacro:drive_wheel_macro robot_namespace="${namespace}"
@@ -64,5 +65,5 @@
     radius="${drive_wheel_radius}"
     length="${drive_wheel_width}"
-    xyz="${drive_wheel_offset_x} ${-drive_wheel_separation/2} ${drive_wheel_offset_z}">
+    xyz="0 ${-drive_wheel_separation/2} 0">
   </xacro:drive_wheel_macro>
   <!-- Left drive wheel -->
@@ -73,5 +74,5 @@
     radius="${drive_wheel_radius}"
     length="${drive_wheel_width}"
-    xyz="${drive_wheel_offset_x} ${drive_wheel_separation/2} ${drive_wheel_offset_z}">
+    xyz="0 ${drive_wheel_separation/2} 0">
   </xacro:drive_wheel_macro>
   <!-- Dummy caster wheel -->
@@ -79,5 +80,6 @@
     parent="base_link"
     prefix="${dummy_caster_wheel_prefix}"
-    xyz="-${dummy_caster_wheel_offset_x} ${dummy_caster_wheel_offset_y} ${drive_wheel_offset_z + dummy_caster_wheel_offset_ground - (drive_wheel_radius - dummy_caster_wheel_radius)}">
+    radius="${dummy_caster_wheel_radius}"
+    xyz="${dummy_caster_wheel_offset_x} ${dummy_caster_wheel_offset_y} ${dummy_caster_wheel_offset_ground - (drive_wheel_radius - dummy_caster_wheel_radius)}">
   </xacro:dummy_caster_wheel_macro>
   <!-- Right laser ranger scanner -->
@@ -85,5 +87,5 @@
     parent="base_link"
     prefix="right">
-    <origin xyz="${base_width/2 + 0.025} -${base_length/2 + 0.025} ${-base_height/2}" rpy="${rad180} 0 ${-rad45}"/>
+    <origin xyz="${chassis_width/2 + (chassis_offset_x + 0.025)} -${chassis_length/2 + 0.025} 0.10" rpy="${rad180} 0 ${-rad45}"/>
   </xacro:hokuyo_macro>
   <!-- Left laser ranger scanner -->
@@ -91,6 +93,12 @@
     parent="base_link"
     prefix="left">
-    <origin xyz="-${base_width/2 + 0.025} ${base_length/2 + 0.025} ${-base_height/2}" rpy="${rad180} 0 ${rad135}"/>
+    <origin xyz="${chassis_offset_x - (chassis_width/2 + 0.025)} ${chassis_length/2 + 0.025} 0.10" rpy="${rad180} 0 ${rad135}"/>
   </xacro:hokuyo_macro>
+  <!-- IMU 0 -->
+  <xacro:imu_macro robot_namespace="${namespace}"
+    parent="base_link"
+    suffix="0">
+    <origin xyz="0 0 0" rpy="0 0 0"/>
+  </xacro:imu_macro>
   <!-- IMU 1 -->
   <xacro:imu_macro robot_namespace="${namespace}"
@@ -99,9 +107,19 @@
     <origin xyz="0 0 0" rpy="0 0 0"/>
   </xacro:imu_macro>
-  <!-- IMU 2 -->
-  <xacro:imu_macro robot_namespace="${namespace}"
-    parent="base_link"
-    suffix="2">
-    <origin xyz="0 0 0" rpy="0 0 0"/>
-  </xacro:imu_macro>
+  <!-- Ground truth (P3D) plugin -->
+  <xacro:if value="${optionals['enable_ground_truth']}">
+    <xacro:p3d_plugin_macro robot_namespace="${namespace}"
+      parent="base_link"
+      update_rate="100"
+      topic_name="odometry/ground_truth"
+      mass="0.00001"
+      body_name="base_footprint"
+      frame_name="world"
+      noise="0"
+      xyz_offset="0 0 0"
+      rpy_offset="0 0 0">
+      <inertia ixx="0.00001" ixy="0" ixz="0" iyy="0.00001" iyz="0" izz="0.00001"/>
+      <origin xyz="0 0 0" rpy="0 0 0"/>
+    </xacro:p3d_plugin_macro>
+  </xacro:if>
 </robot>

File: urdf/plugins/differential_drive_plugin.gazebo.xacro (robot description, xacro)
@@ -1,10 +1,9 @@
 <?xml version="1.0"?>
 <robot xmlns:xacro="http://ros.org/wiki/xacro">
-  <xacro:macro name="differential_drive_macro" params="robot_namespace right_wheel_prefix left_wheel_prefix wheel_separation wheel_diameter wheel_max_torque wheel_max_acceleration">
+  <xacro:macro name="differential_drive_plugin_macro" params="robot_namespace right_wheel_prefix left_wheel_prefix wheel_separation wheel_diameter wheel_max_torque wheel_max_acceleration">
     <gazebo>
       <plugin name="gazebo_ros_diff_drive" filename="libgazebo_ros_diff_drive.so">
         <ros>
           <remapping>odom:=odometry/unfiltered</remapping>
-          <remapping>cmd_vel:=velocity_cmd</remapping>
         </ros>
         <odometry_frame>${robot_namespace}/odom</odometry_frame>
@@ -19,5 +18,5 @@
         <publish_odom_tf>true</publish_odom_tf>
         <publish_wheel_tf>false</publish_wheel_tf>
-        <robot_base_frame>${robot_namespace}/base_footprint</robot_base_frame>
+        <robot_base_frame>${robot_namespace}/base_link</robot_base_frame>
       </plugin>
     </gazebo>

File: urdf/sensors/hokuyo.urdf.xacro (robot description, xacro)
@@ -2,9 +2,4 @@
 <robot xmlns:xacro="http://ros.org/wiki/xacro">
   <xacro:macro name="hokuyo_macro" params="robot_namespace parent prefix *origin">
-    <joint name="${robot_namespace}/${prefix}_hokuyo_joint" type="fixed">
-      <xacro:insert_block name="origin"/>
-      <parent link="${robot_namespace}/${parent}"/>
-      <child link="${robot_namespace}/${prefix}_hokuyo_link"/>
-    </joint>
     <link name="${robot_namespace}/${prefix}_hokuyo_link">
       <visual>
@@ -16,4 +11,9 @@
       </visual>
     </link>
+    <joint name="${robot_namespace}/${prefix}_hokuyo_joint" type="fixed">
+      <xacro:insert_block name="origin"/>
+      <parent link="${robot_namespace}/${parent}"/>
+      <child link="${robot_namespace}/${prefix}_hokuyo_link"/>
+    </joint>
     <!-- Gazebo elements -->
     <gazebo reference="${robot_namespace}/${prefix}_hokuyo_link">

File: urdf/sensors/imu.urdf.xacro (robot description, xacro)
@@ -2,5 +2,11 @@
 <robot xmlns:xacro="http://ros.org/wiki/xacro">
   <xacro:macro name="imu_macro" params="robot_namespace parent suffix *origin">
-    <link name="${robot_namespace}/imu${suffix}_link"/>
+    <link name="${robot_namespace}/imu${suffix}_link">
+      <inertial>
+        <inertia ixx="0.00001" ixy="0.0" ixz="0.0" iyy="0.00001" iyz="0.0" izz="0.00001"/>
+        <mass value="0.0015"/>
+        <origin xyz="0 0 0" rpy="0 0 0"/>
+      </inertial>
+    </link>
     <joint name="${robot_namespace}/imu${suffix}_joint" type="fixed">
       <xacro:insert_block name="origin"/>
@@ -11,12 +17,17 @@
     <!-- Gazebo elements -->
     <gazebo reference="${robot_namespace}/imu${suffix}_link">
+      <gravity>true</gravity>
       <sensor name="${robot_namespace}/imu${suffix}" type="imu">
         <always_on>true</always_on>
-        <visualize>false</visualize>
         <update_rate>100</update_rate>
+        <visualize>true</visualize>
         <plugin name="${robot_namespace}_imu${suffix}_gazebo_ros_imu_sensor" filename="libgazebo_ros_imu_sensor.so">
           <ros>
-            <remapping>~/out:=/${robot_namespace}/imu${suffix}</remapping>
+            <remapping>~/out:=/${robot_namespace}/imu${suffix}/data</remapping>
           </ros>
+          <body_name>${robot_namespace}/imu${suffix}_link</body_name>
+          <gaussian_noise>0.0</gaussian_noise>
+          <xyz_offset>0 0 0</xyz_offset>
+          <rpy_offset>0 0 0</rpy_offset>
           <frame_name>${robot_namespace}/imu${suffix}_link</frame_name>
           <initial_orientation_as_reference>false</initial_orientation_as_reference>

File: urdf/wheels/dummy_caster_wheel.urdf.xacro (robot description, xacro)
@@ -1,5 +1,5 @@
 <?xml version="1.0"?>
 <robot xmlns:xacro="http://ros.org/wiki/xacro">
-  <xacro:macro name="dummy_caster_wheel_macro" params="robot_namespace parent prefix xyz">
+  <xacro:macro name="dummy_caster_wheel_macro" params="robot_namespace parent radius prefix xyz">
     <link name="${robot_namespace}/${prefix}_link">
       <visual>
